File: hardware/GeigerCounter/main.brd (EAGLE design)
At the start: 53.8 x 32.8 mm, 34 parts, among them T4 

Commit message: Fixed PCB.
Parts:
- removed C3: (no value), resistor:C102-054X133
- T5: device transistor:TO126 -> transistor-npn:SOT23
- moved T5 6.11 mm to (44.2, 13.0), flipped to the bottom, turned to 0 degrees
- moved C2 2.29 mm to (85.6, 15.7)
- moved T4 2.17 mm to (73.7, 17.3)
- moved LED1 1.44 mm to (48.5, 7.87)
- moved R12 1.27 mm to (48.0, 14.2), turned to 0 degrees
- moved C5 1.02 mm to (48.8, 31.8), turned to 90 degrees
- moved R2 0.76 mm to (70.6, 16.5)
- moved T7 0.51 mm to (64.0, 9.91)
Connections:
- net N$12: no longer C3.1
- net N$13: now also T5.3; no longer T5.2
- net N$5: now also T5.2; no longer C3.2, T5.1
- net N$9: now also T5.1; no longer T5.3
Routing:
- net N$7: track 112.1 -> 104.4 mm
- net N$5: track 157.8 -> 164.8 mm
- net N$13: track 7.41 -> 3.45 mm
- net N$6: track 2.11 -> 5.39 mm
- net N$12: track 17.0 -> 14.0 mm
- net N$9: track 11.2 -> 8.56 mm
- net N$3: track 2.97 -> 4.13 mm
- net N$4: track 8.47 -> 9.40 mm
- net N$1: track 2.23 -> 3.10 mm
- net N$10: track 11.5 -> 12.2 mm
Other:
- board size 53.8 x 32.8 mm -> 56.1 x 33.8 mm
- board text added: "v1.2"
- board text removed: "v1.1"

Commit message: Built and tested version.
Parts:
- removed SV1(PWM): (no value), con-lstb:MA04-1
- removed T4, T5: (no value), transistor-npn:SOT23
- added C3: (no value), resistor:C050-025X075
- added C6, C7: 330u, resistor:A/3216-18W
- added D2: BAS40, diode:SOT23
- added IC2: (no value), ic-package:DIL08
- C1: device resistor:C050-050X075 -> resistor:C050-025X075
- C2: device resistor:C102-054X133 -> resistor:C3216
- C4: device resistor:C3216 -> resistor:C102-064X133
- C5: value (none) -> 100n; device resistor:E5-8,5 -> resistor:C3216
- IC1: value (none) -> LM358D; device linear:DIL08 -> linear:SO08
- L1: device resistor:TJ5-U1 -> resistor:0207/5V
- R1: device resistor:M1206 -> resistor:0207/5V
- R10, R11, R9: value (none) -> 1k
- R12: value (none) -> 510R
- SP1: value (none) -> 8R; device buzzer:AL60P -> buzzer:KSS1201
- T3: value (none) -> IRF840; device transistor-fet:TO220 -> transistor-power:TO220BV
- moved T2 36.8 mm to (50.8, 14.0)
- moved R1 30.7 mm to (55.9, 21.6), flipped to the top
- moved C2 25.7 mm to (64.5, 30.5), flipped to the bottom, turned to 180 degrees
- moved R7 22.7 mm to (70.5, 15.2), turned to 270 degrees
- moved C4 22.2 mm to (80.4, 17.8), flipped to the top, turned to 90 degrees
- moved C5 20.9 mm to (59.7, 14.0), flipped to the bottom, turned to 270 degrees
- moved SV2(GM) 19.8 mm to (100.9, 14.6), turned to 270 degrees
- moved R5 17.3 mm to (94.5, 9.53), turned to 0 degrees
- moved R2 16.8 mm to (73.7, 33.0), turned to 270 degrees
- moved R8 15.8 mm to (63.5, 17.8), turned to 180 degrees
- moved R9 15.6 mm to (73.7, 3.81), turned to 270 degrees
- moved R6 14.0 mm to (97.1, 19.7), turned to 270 degrees
- moved L1 11.1 mm to (85.1, 31.1), turned to 0 degrees
- moved IC1 10.7 mm to (64.8, 12.7), flipped to the bottom, turned to 270 degrees
- moved T1 9.51 mm to (82.5, 35.6), turned to 90 degrees
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Connections:
- removed net N$14: R1.1, SV1(PWM).3
- removed net N$7: C4.1, C5.+, IC1.8, L1.1, R12.2, R2.2, R8.2, SP1.1, SV1(PWM).4, SV4(POWER).3, T2.3
- new net V+: C2.1, C5.1, C6.+, C7.+, IC1.8, IC2.6, L1.1, R1.2, R12.2, R8.2, SP1.+, SV4(POWER).3
- new net V-: C1.2, C2.2, C3.2, C4.2, C5.2, C6.-, C7.-, IC1.4, IC1.5, IC2.4, R2.1, R3.1, R6.1, R7.1, SV3(OUT).1, SV4(POWER).1, T1.C, T2.2, T3.S, T6.2, T7.2
- net N$10: now also R11.2, T2.1; no longer C1.1, R3.2, R4.1, T4.1
- net N$11: now also IC2.1, IC2.7, IC2.8, R1.1; no longer R2.1, SV1(PWM).2, T4.3
- net N$12: now also C4.1; no longer C2.1
- net N$13: now also C3.1, IC2.5, R3.2, R4.1; no longer SP1.2, T5.3
- net N$15: now also T3.D; no longer T3.2
- net N$16: now also D2.3, T3.G; no longer T2.2, T3.1
- net N$18: now also D2.1, IC2.3, R2.2; no longer R1.2, T2.1
- net N$5: now also C1.1, IC2.2; no longer C1.2, C2.2, C4.2, C5.-, IC1.4, IC1.5, R3.1, R6.1, R7.1, SV1(PWM).1, SV3(OUT).1, SV4(POWER).1, T1.C, T3.3, T4.2, T5.2, T6.2, T7.2
- net N$9: now also SP1.-, T2.3; no longer R11.2, T5.1
Routing:
- net N$5: track 164.8 -> 4.45 mm, vias 6 -> 0
- net N$7: track 104.4 -> 0.00 mm, vias 4 -> 0
- net V+: track 0.00 -> 89.3 mm
- net N$14: track 35.3 -> 0.00 mm
- net V-: track 0.00 -> 26.3 mm, vias 0 -> 2
- net N$8: track 12.0 -> 34.1 mm
- net N$12: track 14.0 -> 33.6 mm
- net N$16: track 7.22 -> 25.7 mm
- net N$18: track 12.2 -> 30.1 mm, vias 0 -> 2
- net N$13: track 3.45 -> 20.9 mm
- net N$11: track 30.8 -> 14.6 mm, vias 2 -> 0
- net N$10: track 12.2 -> 2.14 mm
- net N$17: track 34.3 -> 44.3 mm
- net N$19: track 19.4 -> 10.1 mm
- net N$6: track 5.39 -> 11.8 mm
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- added copper zone on layer 16, net V-
Other:
- board size 56.1 x 33.8 mm -> 60.9 x 38.1 mm
- board text added: "+5V"
- board text added: "G+"
- board text added: "G-"
- board text added: "GND"
- board text added: "HIGH VOLTAGE"
- board text added: "SIGNAL"
- board text added: "V+"
- board text added: "robertgawron.blogspot.com"
- board text added: "v2.1"
- board text removed: "v1.2"

Commit message: Fixed as is on HW model.
Parts:
- C1: value (none) -> 322
- C2: value (none) -> 100n
- C3: value (none) -> 102
- C4: value (none) -> 100n/630V
- D1: value (none) -> 1n4007
- L1: value (none) -> 680m
- R2, R6: value (none) -> 10k
- R3: value (none) -> 30k+1k
- R4: value (none) -> 10M
- R5: value (none) -> 6M8
- R7: value (none) -> 470R
Connections:
- removed net N$18: D2.1, IC2.3, R2.2, T1.B
- new net N$14: D2.1, IC2.2, R2.2, T1.B
- net N$5: now also IC2.3; no longer IC2.2
Routing:
- net N$18: track 30.1 -> 0.00 mm, vias 2 -> 0
- net N$14: track 0.00 -> 18.0 mm, vias 0 -> 2
- net N$5: track 4.45 -> 5.50 mm
Changed lines of the file:
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@@
 <attribute name="VALUE" x="54.5846" y="24.9174" size="1.27" layer="28" ratio="10" rot="MR0"/>
 </element>
-<element name="C3" library="resistor" package="C050-025X075" value="" x="70.485" y="22.86" smashed="yes" rot="R90">
+<element name="C3" library="resistor" package="C050-025X075" value="102" x="70.485" y="22.86" smashed="yes" rot="R90">
 <attribute name="NAME" x="67.564" y="25.781" size="1.27" layer="25" ratio="10" rot="R270"/>
 <attribute name="VALUE" x="73.279" y="19.431" size="1.27" layer="27" ratio="10" rot="R90"/>
 </element>
-<element name="D1" library="diode" package="DO41-10" value="" x="85.725" y="26.035" smashed="yes">
+<element name="D1" library="diode" package="DO41-10" value="1n4007" x="85.725" y="26.035" smashed="yes">
 <attribute name="NAME" x="84.963" y="27.686" size="1.27" layer="25" ratio="10"/>
 <attribute name="VALUE" x="83.693" y="23.241" size="1.27" layer="27" ratio="10"/>
@@
 <attribute name="VALUE" x="43.815" y="13.335" size="1.27" layer="28" rot="MR90"/>
 </element>
-<element name="R6" library="resistor" package="0207/5V" value="" x="97.075" y="19.685" smashed="yes" rot="R270">
+<element name="R6" library="resistor" package="0207/5V" value="10k" x="97.075" y="19.685" smashed="yes" rot="R270">
 <attribute name="NAME" x="94.789" y="20.828" size="1.27" layer="25" ratio="10" rot="R270"/>
 <attribute name="VALUE" x="94.916" y="20.828" size="1.27" layer="27" ratio="10" rot="R270"/>
 </element>
-<element name="R7" library="resistor" package="0207/5V" value="" x="70.485" y="15.24" smashed="yes" rot="R270">
+<element name="R7" library="resistor" package="0207/5V" value="470R" x="70.485" y="15.24" smashed="yes" rot="R270">
 <attribute name="NAME" x="68.199" y="16.002" size="1.27" layer="25" ratio="10" rot="R270"/>
 <attribute name="VALUE" x="68.326" y="16.383" size="1.27" layer="27" ratio="10" rot="R270"/>
@@
 <attribute name="VALUE" x="56.515" y="13.208" size="1.27" layer="28" rot="MR0"/>
 </element>
-<element name="R4" library="resistor" package="0207/5V" value="" x="73.66" y="15.24" smashed="yes" rot="R270">
+<element name="R4" library="resistor" package="0207/5V" value="10M" x="73.66" y="15.24" smashed="yes" rot="R270">
 <attribute name="NAME" x="71.374" y="16.383" size="1.27" layer="25" ratio="10" rot="R270"/>
 <attribute name="VALUE" x="71.501" y="16.383" size="1.27" layer="27" ratio="10" rot="R270"/>
 </element>
-<element name="R3" library="resistor" package="0207/5V" value="" x="73.66" y="22.86" smashed="yes" rot="R270">
+<element name="R3" library="resistor" package="0207/5V" value="30k+1k" x="73.66" y="22.86" smashed="yes" rot="R270">
 <attribute name="NAME" x="75.565" y="21.4376" size="1.27" layer="25" ratio="10" rot="R90"/>
 <attribute name="VALUE" x="71.501" y="24.003" size="1.27" layer="27" ratio="10" rot="R270"/>
@@
 </element>
 <element name="T1" library="transistor" package="SOT23-BEC" value="" x="82.55" y="35.56" rot="MR90"/>
-<element name="R5" library="resistor" package="0207/12" value="" x="94.535" y="9.525" smashed="yes">
+<element name="R5" library="resistor" package="0207/12" value="6M8" x="94.535" y="9.525" smashed="yes">
 <attribute name="NAME" x="93.392" y="7.112" size="1.27" layer="25" ratio="10"/>
 <attribute name="VALUE" x="92.249" y="8.8392" size="1.27" layer="27" ratio="10"/>
@@
 <attribute name="VALUE" x="62.23" y="15.24" size="1.27" layer="28" rot="MR270"/>
 </element>
-<element name="L1" library="resistor" package="0207/5V" value="" x="85.09" y="31.115"/>
-<element name="C4" library="resistor" package="C102-064X133" value="" x="80.375" y="17.78" smashed="yes" rot="R90">
+<element name="L1" library="resistor" package="0207/5V" value="680m" x="85.09" y="31.115"/>
+<element name="C4" library="resistor" package="C102-064X133" value="100n/630V" x="80.375" y="17.78" smashed="yes" rot="R90">
 <attribute name="NAME" x="81.899" y="18.669" size="1.27" layer="25" ratio="10" rot="R90"/>
 <attribute name="VALUE" x="82.28" y="16.256" size="1.27" layer="27" ratio="10" rot="R90"/>
 </element>
-<element name="R2" library="resistor" package="0207/5V" value="" x="73.66" y="33.02" smashed="yes" rot="R270">
+<element name="R2" library="resistor" package="0207/5V" value="10k" x="73.66" y="33.02" smashed="yes" rot="R270">
 <attribute name="NAME" x="74.549" y="33.528" size="1.27" layer="25" ratio="10" rot="R270"/>
 <attribute name="VALUE" x="71.501" y="34.163" size="1.27" layer="27" ratio="10" rot="R270"/>
@@
 <attribute name="VALUE" x="58.674" y="29.21" size="1.27" layer="27" ratio="10"/>
 </element>
-<element name="C1" library="resistor" package="C050-025X075" value="" x="63.5" y="21.59" smashed="yes">
+<element name="C1" library="resistor" package="C050-025X075" value="322" x="63.5" y="21.59" smashed="yes">
 <attribute name="NAME" x="61.976" y="18.796" size="1.27" layer="25" ratio="10"/>
 <attribute name="VALUE" x="60.071" y="18.796" size="1.27" layer="27" ratio="10"/>
@@
 <attribute name="VALUE" x="57.023" y="23.749" size="1.27" layer="27" ratio="10" rot="R180"/>
 </element>
-<element name="C2" library="resistor" package="C3216" value="" x="64.516" y="30.48" smashed="yes" rot="MR180">
+<element name="C2" library="resistor" package="C3216" value="100n" x="64.516" y="30.48" smashed="yes" rot="MR180">
 <attribute name="NAME" x="63.246" y="29.21" size="1.27" layer="26" rot="MR180"/>
 <attribute name="VALUE" x="63.246" y="33.02" size="1.27" layer="28" rot="MR180"/>
@@
 <wire x1="81.77" y1="36.83" x2="81.45" y2="36.51" width="0.6096" layer="16"/>
 </signal>
-<signal name="N$18">
-<contactref element="T1" pad="B"/>
-<contactref element="R2" pad="2"/>
-<contactref element="D2" pad="1"/>
-<contactref element="IC2" pad="3"/>
-<wire x1="60.325" y1="30.48" x2="71.12" y2="30.48" width="0.6096" layer="1"/>
-<via x="60.325" y="30.48" extent="1-16" drill="1" shape="octagon"/>
-<via x="71.12" y="30.48" extent="1-16" drill="1" shape="octagon"/>
-<wire x1="60.325" y1="30.48" x2="60.325" y2="29.21" width="0.6096" layer="16"/>
-<wire x1="60.325" y1="29.21" x2="60.96" y2="28.575" width="0.6096" layer="16"/>
-<wire x1="60.96" y1="28.575" x2="62.23" y2="28.575" width="0.6096" layer="16"/>
-<wire x1="62.23" y1="28.575" x2="63.5" y2="27.305" width="0.6096" layer="16"/>
-<wire x1="63.5" y1="27.305" x2="63.5" y2="26.035" width="0.6096" layer="16"/>
-<wire x1="81.45" y1="34.61" x2="80.965" y2="34.61" width="0.6096" layer="16"/>
-<wire x1="80.965" y1="34.61" x2="80.645" y2="34.29" width="0.6096" layer="16"/>
-<wire x1="80.645" y1="34.29" x2="77.96" y2="34.29" width="0.6096" layer="16"/>
-<wire x1="77.96" y1="34.29" x2="77.64" y2="34.61" width="0.6096" layer="16"/>
-<wire x1="71.12" y1="30.48" x2="73.66" y2="30.48" width="0.6096" layer="16"/>
-<wire x1="73.66" y1="30.48" x2="74.295" y2="30.48" width="0.6096" layer="16"/>
-<wire x1="74.295" y1="30.48" x2="77.47" y2="33.655" width="0.6096" layer="16"/>
-<wire x1="77.47" y1="33.655" x2="77.47" y2="34.44" width="0.6096" layer="16"/>
-<wire x1="77.47" y1="34.44" x2="77.64" y2="34.61" width="0.6096" layer="16"/>
-</signal>
 <signal name="N$22">
 <contactref element="IC1" pad="6"/>
@@
 <signal name="N$5">
 <contactref element="C1" pad="1"/>
+<contactref element="IC2" pad="3"/>
+<wire x1="63.5" y1="26.035" x2="63.5" y2="24.13" width="0.6096" layer="16"/>
+<wire x1="63.5" y1="24.13" x2="60.96" y2="21.59" width="0.6096" layer="16"/>
+</signal>
+<signal name="N$14">
 <contactref element="IC2" pad="2"/>
-<wire x1="60.96" y1="26.035" x2="60.96" y2="21.59" width="0.6096" layer="16"/>
+<contactref element="R2" pad="2"/>
+<contactref element="D2" pad="1"/>
+<contactref element="T1" pad="B"/>
+<wire x1="60.96" y1="26.035" x2="60.96" y2="29.845" width="0.6096" layer="16"/>
+<wire x1="60.96" y1="29.845" x2="60.325" y2="30.48" width="0.6096" layer="16"/>
+<wire x1="60.325" y1="30.48" x2="71.12" y2="30.48" width="0.6096" layer="1"/>
+<wire x1="71.12" y1="30.48" x2="73.66" y2="30.48" width="0.6096" layer="16"/>
+<via x="60.325" y="30.48" extent="1-16" drill="1" shape="octagon"/>
+<via x="71.12" y="30.48" extent="1-16" drill="1" shape="octagon"/>
+<wire x1="77.64" y1="34.61" x2="81.45" y2="34.61" width="0" layer="19" extent="16-16"/>
+<wire x1="73.66" y1="30.48" x2="77.64" y2="34.61" width="0" layer="19" extent="16-16"/>
 </signal>
 </signals>
