File: hardware/tube-connector.brd (EAGLE design)
At the start: 8 parts

Commit message: After first prototype.
Parts:
- moved JP5 28.0 mm to (42.5, 35.0)
- moved U$5 20.2 mm to (35.0, 62.5)
- moved U$6 20.2 mm to (35.0, 27.5)
- moved U$4 20.0 mm to (35.0, 45.0)
- moved JP2 9.01 mm to (12.5, 35.0)
- moved U$2 2.50 mm to (20.0, 62.5)
- moved U$3 2.50 mm to (20.0, 27.5)
Routing:
- net N$4: track 0.00 -> 47.5 mm
- net N$3: track 0.00 -> 47.5 mm
- added copper zone on layer 16, net N$1
- removed copper zone on layer 16, net N$3
- removed copper zone on layer 16, net N$4
Other:
- board outline added: 40 x 70 mm
