File: hardware/GeigerMuller_shield.brd (EAGLE design)
At the start: 28 parts

Commit message: Fixed resistor value.
Parts:
- R5: value 10k -> 220R
Changed lines of the file:
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@@
 <element name="C5" library="resistor" package="C0805K" value="10n" x="49.53" y="24.13" rot="MR90"/>
 <element name="C6" library="resistor" package="C0805K" value="10n" x="52.07" y="24.13" rot="MR90"/>
-<element name="R5" library="resistor" package="0207/10" value="10k" x="35.56" y="13.97" rot="MR270"/>
+<element name="R5" library="resistor" package="0207/10" value="220R" x="35.56" y="13.97" rot="MR270"/>
 <element name="GM_SIGNAL" library="con-molex" package="7395-02" value="22-05-7028-02" x="55.245" y="31.115" rot="R90">
 <attribute name="MF" value="" x="55.245" y="31.115" size="1.778" layer="27" rot="R90" display="off"/>

Commit message: Fixes in arduino shield.
Parts:
- removed RESET1, RESET2: (no value), switch-omron:B3F-10XX
- added DOWN, UP: (no value), switch-omron:B3F-10XX
- moved RESET 44.2 mm to (21.0, 5.71)
- moved R1 11.5 mm to (26.7, 25.4)
- moved R3 11.5 mm to (26.7, 30.5)
- moved C1 11.5 mm to (27.9, 19.1)
- moved C2 11.5 mm to (29.2, 25.4)
- moved C3 11.5 mm to (27.9, 36.8)
- moved C4 11.5 mm to (29.2, 30.5)
- moved R2 11.5 mm to (27.9, 21.6)
- moved R4 11.5 mm to (27.9, 34.3)
- moved JP1 7.73 mm to (35.6, 26.7)
- moved C7 4.26 mm to (45.7, 36.2)
- moved J8 2.54 mm to (52.1, 40.0), turned to 180 degrees
- moved R5 1.90 mm to (35.6, 15.9), flipped to the top
Connections:
- net GND: now also DOWN.4, UP.4; no longer RESET1.4, RESET2.4
- net LCD_CS: now also J8.4; no longer J8.2
- net LCD_DIN: now also J8.2; no longer J8.4
- net LCD_RST: now also J8.5; no longer J8.1
- net LCD_SCLK: now also J8.1; no longer J8.5
- net N$17: now also DOWN.2; no longer RESET2.2
- net N$5: now also UP.2; no longer RESET1.2
Routing:
- net RESET: track 81.8 -> 20.2 mm
- net +5V: track 142.0 -> 88.2 mm
- net LCD_BACKLIGHT: track 41.7 -> 19.4 mm
- net BUTTON_2: track 31.8 -> 20.9 mm
- net BUTTON_1: track 45.9 -> 37.8 mm
- net N$8: track 9.20 -> 3.18 mm
- net LCD_DC: track 9.31 -> 12.9 mm
- net LCD_CS: track 9.31 -> 12.9 mm
- net LCD_SCLK: track 9.31 -> 12.9 mm
- net LCD_RST: track 9.31 -> 12.9 mm
- net LCD_DIN: track 9.31 -> 12.9 mm
- net 3V3: track 6.35 -> 8.25 mm
Other:
- board outline added: 51 x 53 mm
