File: hardware/GeigerMuller_shield.sch (EAGLE design)
At the start: 28 parts

Commit message: Fixed resistor value.
Parts:
- R5: value 10k -> 220R
Changed lines of the file:
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@@
 <setting verticaltext="up"/>
 </settings>
-<grid distance="0.1" unitdist="inch" unit="inch" style="lines" multiple="1" display="yes" altdistance="0.01" altunitdist="inch" altunit="inch"/>
+<grid distance="0.1" unitdist="inch" unit="inch" style="lines" multiple="1" display="no" altdistance="0.01" altunitdist="inch" altunit="inch"/>
 <layers>
 <layer number="1" name="Top" color="4" fill="1" visible="no" active="no"/>
@@
 <part name="C5" library="resistor" deviceset="C-EU" device="C0805K" value="10n"/>
 <part name="C6" library="resistor" deviceset="C-EU" device="C0805K" value="10n"/>
-<part name="R5" library="resistor" deviceset="R-EU_" device="0207/10" value="10k"/>
+<part name="R5" library="resistor" deviceset="R-EU_" device="0207/10" value="220R"/>
 <part name="GM_SIGNAL" library="con-molex" deviceset="22-?-02" device="05-7028"/>
 <part name="GND13" library="supply1" deviceset="GND" device=""/>

Commit message: Fixes in arduino shield.
Parts:
- renumbered RESET1 to UP, RESET2 to DOWN
Connections:
- net LCD_CS: now also J8.4; no longer J8.2
- net LCD_DIN: now also J8.2; no longer J8.4
- net LCD_RST: now also J8.5; no longer J8.1
- net LCD_SCLK: now also J8.1; no longer J8.5
Changed lines of the file:
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@@
 <part name="GND5" library="supply1" deviceset="GND" device=""/>
 <part name="+5V" library="supply1" deviceset="+5V" device=""/>
-<part name="RESET1" library="switch-omron" deviceset="10-XX" device=""/>
+<part name="UP" library="switch-omron" deviceset="10-XX" device=""/>
 <part name="C1" library="resistor" deviceset="C-EU" device="C0805K" value="10n"/>
 <part name="C2" library="resistor" deviceset="C-EU" device="C0805K" value="100n"/>
@@
 <part name="GND8" library="supply1" deviceset="GND" device=""/>
 <part name="P+3" library="supply1" deviceset="+5V" device=""/>
-<part name="RESET2" library="switch-omron" deviceset="10-XX" device=""/>
+<part name="DOWN" library="switch-omron" deviceset="10-XX" device=""/>
 <part name="C3" library="resistor" deviceset="C-EU" device="C0805K" value="10n"/>
 <part name="C4" library="resistor" deviceset="C-EU" device="C0805K" value="100n"/>
@@
 <instance part="GND5" gate="1" x="165.1" y="76.2"/>
 <instance part="+5V" gate="1" x="165.1" y="121.92"/>
-<instance part="RESET1" gate="1" x="162.56" y="86.36"/>
+<instance part="UP" gate="1" x="162.56" y="86.36"/>
 <instance part="C1" gate="G$1" x="180.34" y="88.9"/>
 <instance part="C2" gate="G$1" x="172.72" y="111.76"/>
@@
 <instance part="GND8" gate="1" x="208.28" y="76.2"/>
 <instance part="P+3" gate="1" x="208.28" y="121.92"/>
-<instance part="RESET2" gate="1" x="205.74" y="86.36"/>
+<instance part="DOWN" gate="1" x="205.74" y="86.36"/>
 <instance part="C3" gate="G$1" x="223.52" y="88.9"/>
 <instance part="C4" gate="G$1" x="215.9" y="111.76"/>
@@
 <segment>
 <pinref part="GND5" gate="1" pin="GND"/>
-<pinref part="RESET1" gate="1" pin="P1"/>
+<pinref part="UP" gate="1" pin="P1"/>
 <wire x1="165.1" y1="78.74" x2="165.1" y2="81.28" width="0.1524" layer="91"/>
 </segment>
@@
 <segment>
 <pinref part="GND8" gate="1" pin="GND"/>
-<pinref part="RESET2" gate="1" pin="P1"/>
+<pinref part="DOWN" gate="1" pin="P1"/>
 <wire x1="208.28" y1="78.74" x2="208.28" y2="81.28" width="0.1524" layer="91"/>
 </segment>
@@
 </segment>
 <segment>
-<pinref part="J8" gate="A" pin="1"/>
-<wire x1="157.48" y1="58.42" x2="157.48" y2="30.48" width="0.1524" layer="91"/>
-<wire x1="157.48" y1="30.48" x2="187.96" y2="30.48" width="0.1524" layer="91"/>
+<wire x1="167.64" y1="30.48" x2="187.96" y2="30.48" width="0.1524" layer="91"/>
 <label x="177.8" y="30.48" size="1.778" layer="95"/>
+<pinref part="J8" gate="A" pin="5"/>
+<wire x1="167.64" y1="30.48" x2="167.64" y2="58.42" width="0.1524" layer="91"/>
 </segment>
 </net>
@@
 </segment>
 <segment>
-<pinref part="J8" gate="A" pin="2"/>
-<wire x1="160.02" y1="58.42" x2="160.02" y2="33.02" width="0.1524" layer="91"/>
-<wire x1="160.02" y1="33.02" x2="187.96" y2="33.02" width="0.1524" layer="91"/>
+<wire x1="165.1" y1="33.02" x2="187.96" y2="33.02" width="0.1524" layer="91"/>
 <label x="177.8" y="33.02" size="1.778" layer="95"/>
+<pinref part="J8" gate="A" pin="4"/>
+<wire x1="165.1" y1="33.02" x2="165.1" y2="58.42" width="0.1524" layer="91"/>
 </segment>
 </net>
@@
 </segment>
 <segment>
-<pinref part="J8" gate="A" pin="3"/>
-<wire x1="162.56" y1="58.42" x2="162.56" y2="35.56" width="0.1524" layer="91"/>
 <wire x1="162.56" y1="35.56" x2="187.96" y2="35.56" width="0.1524" layer="91"/>
 <label x="177.8" y="35.56" size="1.778" layer="95"/>
+<pinref part="J8" gate="A" pin="3"/>
+<wire x1="162.56" y1="35.56" x2="162.56" y2="58.42" width="0.1524" layer="91"/>
 </segment>
 </net>
@@
 </segment>
 <segment>
-<pinref part="J8" gate="A" pin="4"/>
-<wire x1="165.1" y1="58.42" x2="165.1" y2="38.1" width="0.1524" layer="91"/>
-<wire x1="165.1" y1="38.1" x2="187.96" y2="38.1" width="0.1524" layer="91"/>
+<wire x1="160.02" y1="38.1" x2="187.96" y2="38.1" width="0.1524" layer="91"/>
 <label x="177.8" y="38.1" size="1.778" layer="95"/>
+<pinref part="J8" gate="A" pin="2"/>
+<wire x1="160.02" y1="38.1" x2="160.02" y2="58.42" width="0.1524" layer="91"/>
 </segment>
 </net>
@@
 </segment>
 <segment>
-<pinref part="J8" gate="A" pin="5"/>
-<wire x1="167.64" y1="58.42" x2="167.64" y2="40.64" width="0.1524" layer="91"/>
-<wire x1="167.64" y1="40.64" x2="187.96" y2="40.64" width="0.1524" layer="91"/>
+<wire x1="157.48" y1="40.64" x2="187.96" y2="40.64" width="0.1524" layer="91"/>
 <label x="177.8" y="40.64" size="1.778" layer="95"/>
+<pinref part="J8" gate="A" pin="1"/>
+<wire x1="157.48" y1="40.64" x2="157.48" y2="58.42" width="0.1524" layer="91"/>
 </segment>
 </net>
@@
 <net name="N$5" class="0">
 <segment>
-<pinref part="RESET1" gate="1" pin="S1"/>
+<pinref part="UP" gate="1" pin="S1"/>
 <pinref part="R1" gate="G$1" pin="1"/>
 <wire x1="165.1" y1="91.44" x2="165.1" y2="93.98" width="0.1524" layer="91"/>
@@
 <net name="N$17" class="0">
 <segment>
-<pinref part="RESET2" gate="1" pin="S1"/>
+<pinref part="DOWN" gate="1" pin="S1"/>
 <pinref part="R3" gate="G$1" pin="1"/>
 <wire x1="208.28" y1="91.44" x2="208.28" y2="93.98" width="0.1524" layer="91"/>
