File: kicad/main.sch (KiCad schematic (older format))
At the start: 34 parts, among them IC2 LM358D, IC3 MC34063AD, J1 Power, J2 GM Tube, Q1 IRF840, Q2 BC558, Q3 BC848SMD, Q4 BC848SMD

Commit message: even more missing files added
Parts:
- added U? (x2): 74469, symbol 74xx:74469
Connections:
- wire segments 140 -> 142
Changed lines of the file:
@@
 EESchema Schematic File Version 4
+LIBS:main-cache
 EELAYER 26 0
 EELAYER END
@@
 Wire Wire Line
 	1950 3950 1950 2900
-Wire Wire Line
-	1750 2900 1950 2900
 Connection ~ 1950 2900
 Wire Wire Line
@@
 Wire Wire Line
 	6100 4100 6250 4100
+$Comp
+L power:PWR_FLAG #FLG?
+U 1 1 5BA8EA25
+P 1850 2700
+F 0 "#FLG?" H 1850 2775 50  0001 C CNN
+F 1 "PWR_FLAG" H 1850 2874 50  0000 C CNN
+F 2 "" H 1850 2700 50  0001 C CNN
+F 3 "~" H 1850 2700 50  0001 C CNN
+	1    1850 2700
+	1    0    0    -1
+$EndComp
+Wire Wire Line
+	1850 2700 1850 2900
+Wire Wire Line
+	1750 2900 1850 2900
+Connection ~ 1850 2900
+Wire Wire Line
+	1850 2900 1950 2900
+$Comp
+L 74xx:74469 U?
+U 1 1 5BA9A521
+P 3050 1200
+F 0 "U?" H 3050 2278 50  0000 C CNN
+F 1 "74469" H 3050 2187 50  0000 C CNN
+F 2 "" H 3050 1200 50  0001 C CNN
+F 3 "http://www.ti.com/lit/gpn/sn74469" H 3050 1200 50  0001 C CNN
+	1    3050 1200
+	1    0    0    -1
+$EndComp
+$Comp
+L 74xx:74469 U?
+U 1 1 5BAA05AC
+P 5600 1300
+F 0 "U?" H 5600 2378 50  0000 C CNN
+F 1 "74469" H 5600 2287 50  0000 C CNN
+F 2 "" H 5600 1300 50  0001 C CNN
+F 3 "http://www.ti.com/lit/gpn/sn74469" H 5600 1300 50  0001 C CNN
+	1    5600 1300
+	1    0    0    -1
+$EndComp
 $EndSCHEMATC

Commit message: elements placement fix
Parts:
- removed Q2: BC558, TO_SOT_Packages_SMD:SOT-23, symbol Transistor_BJT:BC558
- removed U? (x2): 74469, symbol 74xx:74469
- added Q2: BC808, TO_SOT_Packages_SMD:SOT-23, symbol Transistor_BJT:BC808
- D3: footprint Diodes_THT:D_A-405_P2.54mm_Vertical_AnodeUp -> LEDs:LED_D3.0mm
- J1: value 22-?-0205-7028 -> Power
- J2: value 22-?-0205-7028 -> GM Tube
Connections:
- wire segments 142 -> 146
Changed lines of the file:
@@
 	1750 4200 1750 5400
 Wire Wire Line
-	1750 5400 1900 5400
+	1750 5400 1800 5400
 Wire Wire Line
 	2350 4400 2350 4500
@@
 P 1550 4200
 F 0 "J1" H 1650 4170 51  0000 L BNN
-F 1 "Power" H 1520 4255 59  0000 L BNN
+F 1 "Power" H 1520 4255 59  0001 L BNN
 F 2 "Pin_Headers:Pin_Header_Angled_1x02_Pitch2.54mm" H 1550 4200 50  0001 C CNN
 F 3 "" H 1550 4200 50  0001 C CNN
@@
 P 1550 4000
 F 0 "J1" H 1650 3970 51  0000 L BNN
-F 1 "22-?-0205-7028" H 1520 4055 59  0001 L BNN
+F 1 "Power" H 1520 4055 59  0001 L BNN
 F 2 "Pin_Headers:Pin_Header_Angled_1x02_Pitch2.54mm" H 1550 4000 50  0001 C CNN
 F 3 "" H 1550 4000 50  0001 C CNN
@@
 P 8400 4050
 F 0 "J2" H 8500 4020 51  0000 L BNN
-F 1 "GM Tube" H 8370 4105 59  0000 L BNN
+F 1 "GM Tube" H 8370 4105 59  0001 L BNN
 F 2 "Pin_Headers:Pin_Header_Angled_1x02_Pitch2.54mm" H 8400 4050 50  0001 C CNN
 F 3 "" H 8400 4050 50  0001 C CNN
@@
 P 8400 4150
 F 0 "J2" H 8500 4120 51  0000 L BNN
-F 1 "22-?-0205-7028" H 8370 4205 59  0001 L BNN
+F 1 "GM Tube" H 8370 4205 59  0001 L BNN
 F 2 "Pin_Headers:Pin_Header_Angled_1x02_Pitch2.54mm" H 8400 4150 50  0001 C CNN
 F 3 "" H 8400 4150 50  0001 C CNN
@@
 $EndComp
 Wire Notes Line
-	1250 2500 3300 2500
-Wire Notes Line
-	3300 2500 3300 5800
+	1250 2200 3300 2200
+Wire Notes Line
+	3300 2200 3300 5800
 Wire Notes Line
 	3300 5800 1250 5800
 Wire Notes Line
-	1250 5800 1250 2500
+	1250 5800 1250 2200
 Wire Notes Line
 	3400 5800 7500 5800
 Wire Notes Line
-	7500 5800 7500 2500
-Wire Notes Line
-	7500 2500 3400 2500
-Wire Notes Line
-	3400 2500 3400 5800
+	7500 5800 7500 2200
+Wire Notes Line
+	7500 2200 3400 2200
+Wire Notes Line
+	3400 2200 3400 5800
 Wire Notes Line
 	8900 5800 12100 5800
 Wire Notes Line
-	12100 5800 12100 2500
-Wire Notes Line
-	12100 2500 8900 2500
-Wire Notes Line
-	8900 2500 8900 5800
-Wire Notes Line
-	7600 2500 7600 5800
+	12100 5800 12100 2200
+Wire Notes Line
+	12100 2200 8900 2200
+Wire Notes Line
+	8900 2200 8900 5800
+Wire Notes Line
+	7600 2200 7600 5800
 Wire Notes Line
 	7600 5800 8800 5800
 Wire Notes Line
-	8800 5800 8800 2500
-Wire Notes Line
-	8800 2500 7600 2500
-Text Notes 2150 2700 0    150  ~ 0
+	8800 5800 8800 2200
+Wire Notes Line
+	8800 2200 7600 2200
+Text Notes 1500 2500 0    150  ~ 0
 Power supply
-Text Notes 5600 2700 0    150  ~ 0
+Text Notes 4100 2500 0    150  ~ 0
 5V/400V DC/DC converter
-Text Notes 8200 2700 0    150  ~ 0
+Text Notes 7700 2750 0    150  ~ 0
 GM \ndetector
-Text Notes 10800 2700 0    150  ~ 0
+Text Notes 10100 2500 0    150  ~ 0
 Output
 $Comp
@@
 Wire Wire Line
 	9100 5400 10650 5400
-$Comp
-L Transistor_BJT:BC558 Q2
-U 1 1 5BA34A22
-P 5050 5000
-F 0 "Q2" H 5241 4954 50  0000 L CNN
-F 1 "BC558" H 5241 5045 50  0000 L CNN
-F 2 "TO_SOT_Packages_SMD:SOT-23" H 5250 4925 50  0001 L CIN
-F 3 "http://www.fairchildsemi.com/ds/BC/BC557.pdf" H 5050 5000 50  0001 L CNN
-	1    5050 5000
-	1    0    0    1
-$EndComp
 Wire Wire Line
 	4600 5000 4850 5000
@@
 F 0 "D3" V 10688 3583 50  0000 R CNN
 F 1 "LED" V 10597 3583 50  0000 R CNN
-F 2 "Diodes_THT:D_A-405_P2.54mm_Vertical_AnodeUp" H 10650 3700 50  0001 C CNN
+F 2 "LEDs:LED_D3.0mm" H 10650 3700 50  0001 C CNN
 F 3 "~" H 10650 3700 50  0001 C CNN
 	1    10650 3700
@@
 	6100 4100 6250 4100
 $Comp
-L power:PWR_FLAG #FLG?
+L power:PWR_FLAG #FLG0101
 U 1 1 5BA8EA25
-P 1850 2700
-F 0 "#FLG?" H 1850 2775 50  0001 C CNN
-F 1 "PWR_FLAG" H 1850 2874 50  0000 C CNN
-F 2 "" H 1850 2700 50  0001 C CNN
-F 3 "~" H 1850 2700 50  0001 C CNN
-	1    1850 2700
-	1    0    0    -1
-$EndComp
-Wire Wire Line
-	1850 2700 1850 2900
+P 1850 2800
+F 0 "#FLG0101" H 1850 2875 50  0001 C CNN
+F 1 "PWR_FLAG" H 1850 2974 50  0000 C CNN
+F 2 "" H 1850 2800 50  0001 C CNN
+F 3 "~" H 1850 2800 50  0001 C CNN
+	1    1850 2800
+	1    0    0    -1
+$EndComp
+Wire Wire Line
+	1850 2800 1850 2900
 Wire Wire Line
 	1750 2900 1850 2900
@@
 	1850 2900 1950 2900
 $Comp
-L 74xx:74469 U?
-U 1 1 5BA9A521
-P 3050 1200
-F 0 "U?" H 3050 2278 50  0000 C CNN
-F 1 "74469" H 3050 2187 50  0000 C CNN
-F 2 "" H 3050 1200 50  0001 C CNN
-F 3 "http://www.ti.com/lit/gpn/sn74469" H 3050 1200 50  0001 C CNN
-	1    3050 1200
-	1    0    0    -1
-$EndComp
-$Comp
-L 74xx:74469 U?
-U 1 1 5BAA05AC
-P 5600 1300
-F 0 "U?" H 5600 2378 50  0000 C CNN
-F 1 "74469" H 5600 2287 50  0000 C CNN
-F 2 "" H 5600 1300 50  0001 C CNN
-F 3 "http://www.ti.com/lit/gpn/sn74469" H 5600 1300 50  0001 C CNN
-	1    5600 1300
-	1    0    0    -1
+L power:PWR_FLAG #FLG0102
+U 1 1 5BAA09D1
+P 1450 5500
+F 0 "#FLG0102" H 1450 5575 50  0001 C CNN
+F 1 "PWR_FLAG" H 1450 5674 50  0000 C CNN
+F 2 "" H 1450 5500 50  0001 C CNN
+F 3 "~" H 1450 5500 50  0001 C CNN
+	1    1450 5500
+	1    0    0    -1
+$EndComp
+Wire Wire Line
+	1450 5500 1450 5700
+Wire Wire Line
+	1450 5700 1800 5700
+Wire Wire Line
+	1800 5700 1800 5400
+Connection ~ 1800 5400
+Wire Wire Line
+	1800 5400 1900 5400
+$Comp
+L Transistor_BJT:BC808 Q2
+U 1 1 5BAA796E
+P 5050 5000
+F 0 "Q2" H 5241 4954 50  0000 L CNN
+F 1 "BC808" H 5241 5045 50  0000 L CNN
+F 2 "TO_SOT_Packages_SMD:SOT-23" H 5250 4925 50  0001 L CIN
+F 3 "http://www.fairchildsemi.com/ds/BC/BC807.pdf" H 5050 5000 50  0001 L CNN
+	1    5050 5000
+	1    0    0    1
 $EndComp
 $EndSCHEMATC

Commit message: drc check ok
Parts:
- removed Q2: BC808, TO_SOT_Packages_SMD:SOT-23, symbol Transistor_BJT:BC808
- added Q2: Q_PNP_BEC, TO_SOT_Packages_SMD:SOT-23, symbol Device:Q_PNP_BEC
Changed lines of the file:
@@
 	1800 5400 1900 5400
 $Comp
-L Transistor_BJT:BC808 Q2
-U 1 1 5BAA796E
+L Device:Q_PNP_BEC Q2
+U 1 1 5BB1EC0F
 P 5050 5000
-F 0 "Q2" H 5241 4954 50  0000 L CNN
-F 1 "BC808" H 5241 5045 50  0000 L CNN
-F 2 "TO_SOT_Packages_SMD:SOT-23" H 5250 4925 50  0001 L CIN
-F 3 "http://www.fairchildsemi.com/ds/BC/BC807.pdf" H 5050 5000 50  0001 L CNN
+F 0 "Q2" H 5241 5046 50  0000 L CNN
+F 1 "Q_PNP_BEC" H 5241 4955 50  0000 L CNN
+F 2 "TO_SOT_Packages_SMD:SOT-23" H 5250 5100 50  0001 C CNN
+F 3 "~" H 5050 5000 50  0001 C CNN
 	1    5050 5000
-	1    0    0    1
+	1    0    0    -1
 $EndComp
 $EndSCHEMATC
