File: kicad/mainboard/main.kicad_pcb (KiCad board)
At the start: 2 copper layers, 55 x 45 mm, 42 parts, among them IC2 LM358D, IC3 MC34063AD, J1 Conn_01x02_Male, J2 Conn_01x02_Male, J3 Conn_01x02_Male, J4 Conn_01x03_Male, J5 Conn_01x02_Male, Q1 IRF840, Q2 Q_PNP_BEC, Q3 BC848SMD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

Commit message: new hw ready to be send to pcb company
Parts:
- removed the REF** at (125.0, 90.0)
- removed the REF** at (125.0, 125.0)
- added REF**: MountingHole_3.5mm_Pad, Mounting_Holes:MountingHole_3.5mm_Pad, F.Cu at (135.0, 85.0)
- added REF**: MountingHole_3.5mm_Pad, Mounting_Holes:MountingHole_3.5mm_Pad, F.Cu at (135.0, 125.0)
- added REF**: MountingHole_3.5mm_Pad, Mounting_Holes:MountingHole_3.5mm_Pad, F.Cu at (170.0, 85.0)
- C5: footprint Capacitor_THT:C_Rect_L13.0mm_W6.5mm_P7.50mm_P10.00mm -> Capacitors_THT:C_Rect_L13.5mm_W5.0mm_P10.00mm_FKS3_FKP3_MKS4
- J1: footprint Connector_PinHeader_2.54mm:PinHeader_1x02_P2.54mm_Horizontal -> GeigerCounter:GeigerCounterPinHeader_1x02_P2.54mm_Horizontal
- J2 GM+: renamed from J2; footprint Connector_PinHeader_2.54mm:PinHeader_1x02_P2.54mm_Horizontal -> GeigerCounter:GeigerCounterPinHeader_1x02_P2.54mm_Horizontal
- J3 GM-: renamed from J3; footprint Connector_PinHeader_2.54mm:PinHeader_1x02_P2.54mm_Horizontal -> GeigerCounter:GeigerCounterPinHeader_1x02_P2.54mm_Horizontal
- moved C8 19.1 mm to (154.3, 95.2)
- moved D3 9.55 mm to (142.9, 124.5)
- moved Q3 8.28 mm to (146.1, 122.6)
- moved J5 8.28 mm to (148.0, 126.4)
- moved J4 8.28 mm to (154.3, 126.4)
- moved Q4 8.28 mm to (155.3, 121.8)
- moved R11 8.28 mm to (149.5, 121.8)
- moved R12 8.28 mm to (152.1, 121.8)
- moved R14 8.28 mm to (159.7, 121.8)
- moved R7 7.24 mm to (163.8, 117.5), turned to 270 degrees
- moved R13 7.01 mm to (139.7, 119.4)
- moved D4 5.46 mm to (166.4, 118.1), turned to 90 degrees
- moved Q2 5.36 mm to (155.7, 85.1)
- moved D1 4.96 mm to (151.3, 85.1)
- moved C7 3.84 mm to (139.1, 106.2)
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Connections:
- C8 pad 1: Net-(C3-Pad1) -> Net-(C8-Pad1)
- C9 pad 1: Net-(C9-Pad1) -> Net-(C8-Pad1)
- JP1 pad 2: Net-(C9-Pad1) -> Net-(C8-Pad1)
- L1 pad 1: Net-(C9-Pad1) -> Net-(C8-Pad1)
Routing:
- net Net-(C3-Pad1): track 57.2 -> 74.0 mm
- net Net-(IC2-Pad1): track 10.2 -> 24.3 mm
- net Net-(D1-Pad2): track 9.50 -> 22.3 mm
- net Net-(D1-Pad1): track 15.4 -> 26.5 mm
- net Net-(D4-Pad1): track 23.7 -> 34.4 mm
- net Net-(C8-Pad1): track 0.00 -> 9.25 mm
- net Net-(IC3-Pad1): track 18.6 -> 24.4 mm
- net Net-(R4-Pad1): track 0.00 -> 2.54 mm
- net Net-(Q3-Pad1): track 1.94 -> 3.75 mm
- net Net-(IC2-Pad2): track 7.37 -> 8.87 mm
- net Net-(D3-Pad1): track 4.23 -> 2.96 mm
- net Net-(D3-Pad2): track 2.84 -> 3.78 mm
- net Net-(D2-Pad2): track 12.4 -> 11.6 mm
- net GND: vias 3 -> 6
Other:
- board size 55 x 45 mm -> 45 x 50 mm
- board text added: "Geiger Counter"
- board text added: "HIGH VOLTAGE!"
- board text added: "IC out"
- board text added: "IC out V+ selector"
- board text added: "power supply"
- board text added: "rev2.2"
- board text removed: "G+"
- board text removed: "G-"
- board text removed: "Geiger Muller Counter"
- board text removed: "HIGH VOLTAGE!!"
- board text removed: "rev2.3"
