File: hardware/kicad/mainboard/main.kicad_pcb (KiCad board)
At the start: 2 copper layers, 45 x 50 mm, 43 parts, among them IC2 LM358D, IC3 MC34063AD, J1 Conn_01x02_Male, J2 GM+ Conn_01x02_Male, J3 GM- Conn_01x02_Male, J4 Conn_01x03_Male, J5 Conn_01x02_Male, Q1 IRF840, Q2 Q_PNP_BEC, Q3 BC848SMD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

Commit message: fixes after hw tests
Parts:
- removed J2 GM+: Conn_01x02_Male, GeigerCounter:GeigerCounterPinHeader_1x02_P2.54mm_Horizontal
- removed J3 GM-: Conn_01x02_Male, GeigerCounter:GeigerCounterPinHeader_1x02_P2.54mm_Horizontal
- added GM_minus1: Conn_01x02_Male, Pin_Headers:Pin_Header_Straight_1x02_Pitch2.54mm, F.Cu at (170.2, 114.8)
- added GM_plus1: Conn_01x02_Male, Pin_Headers:Pin_Header_Straight_1x02_Pitch2.54mm, F.Cu at (170.2, 104.1)
- C1: value 32n -> not mounted
- C2: value 32n -> 3n2
- C7: value 330u -> 10u 6V3
- J1: footprint GeigerCounter:GeigerCounterPinHeader_1x02_P2.54mm_Horizontal -> Pin_Headers:Pin_Header_Straight_1x02_Pitch2.54mm
- J4: footprint Connector_PinHeader_2.54mm:PinHeader_1x03_P2.54mm_Vertical -> Pin_Headers:Pin_Header_Straight_1x03_Pitch2.54mm
- J5: footprint Connector_PinHeader_2.54mm:PinHeader_1x02_P2.54mm_Vertical -> Pin_Headers:Pin_Header_Straight_1x02_Pitch2.54mm
- Q2: value Q_PNP_BEC -> BC859
- Q3, Q4: value BC848SMD -> BC848
- R13: value 510R -> 470R
- R8: value ? -> 10k
Connections:
- Q2 pad 2: GND -> Net-(D1-Pad1)
- Q2 pad 3: Net-(D1-Pad1) -> GND
Routing:
- net Net-(D1-Pad1): track 26.5 -> 24.1 mm
- net Net-(GM_plus1-Pad1): track 6.24 -> 6.88 mm
