File: hardware/kicad/mainboard/main.sch (KiCad schematic (older format))
At the start: 39 parts, among them IC2 LM358D, IC3 MC34063AD, J1 Conn_01x02_Male, J2 Conn_01x02_Male, J3 Conn_01x02_Male, J4 Conn_01x03_Male, J5 Conn_01x02_Male, Q1 IRF840, Q2 Q_PNP_BEC, Q3 BC848SMD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

Commit message: fixes after hw tests
Parts:
- removed Q2: Q_PNP_BEC, TO_SOT_Packages_SMD:SOT-23, symbol Device:Q_PNP_BEC
- removed Q3, Q4: BC848SMD, TO_SOT_Packages_SMD:SOT-23, symbol main-eagle-import:BC848SMD
- added Q2: BC859, TO_SOT_Packages_SMD:SOT-23, symbol Transistor_BJT:BC859
- added Q3, Q4: BC848, TO_SOT_Packages_SMD:SOT-23, symbol Transistor_BJT:BC848
- C1: value 32n -> not mounted
- C2: value 32n -> 3n2
- C7: value 330u -> 10u 6V3
- GM_minus: renamed from J3; footprint Connector_PinHeader_2.54mm:PinHeader_1x02_P2.54mm_Horizontal -> Pin_Headers:Pin_Header_Straight_1x02_Pitch2.54mm
- GM_plus: renamed from J2; footprint Connector_PinHeader_2.54mm:PinHeader_1x02_P2.54mm_Horizontal -> Pin_Headers:Pin_Header_Straight_1x02_Pitch2.54mm
- J1: footprint Connector_PinHeader_2.54mm:PinHeader_1x02_P2.54mm_Horizontal -> Pin_Headers:Pin_Header_Straight_1x02_Pitch2.54mm
- J4: footprint Connector_PinHeader_2.54mm:PinHeader_1x03_P2.54mm_Vertical -> Pin_Headers:Pin_Header_Straight_1x03_Pitch2.54mm
- J5: footprint Connector_PinHeader_2.54mm:PinHeader_1x02_P2.54mm_Vertical -> Pin_Headers:Pin_Header_Straight_1x02_Pitch2.54mm
- R13: value 510R -> 470R
- R8: value ? -> 10k
Other:
- moved on the sheet: D3, J4, R11, R12, R13, R14
