File: Hardware/mainboard/main.kicad_pcb (KiCad board)
At the start: 2 copper layers, 45 x 50 mm, 43 parts, among them IC2 LM358D, IC3 MC34063AD, J1 Conn_01x02_Male, J4 Conn_01x03_Male, J5 Conn_01x02_Male, Q1 IRF840, Q2 BC859, Q3 BC848, Q4 BC848

Commit message: use kicad elments (after eagle to kicad transition)
Parts:
- turned R1 to 90 degrees
- turned R11 to 90 degrees
- turned R12 to 90 degrees
- turned R14 to 180 degrees
- turned R8 to 0 degrees
- turned R9 to 180 degrees
Connections:
- R1 pad 1: GND -> Net-(D1-Pad2)
- R1 pad 2: Net-(D1-Pad2) -> GND
- R11 pad 1: Net-(IC2-Pad1) -> Net-(Q3-Pad1)
- R11 pad 2: Net-(Q3-Pad1) -> Net-(IC2-Pad1)
- R12 pad 1: Net-(IC2-Pad1) -> Net-(Q4-Pad1)
- R12 pad 2: Net-(Q4-Pad1) -> Net-(IC2-Pad1)
- R14 pad 1: Net-(J4-Pad2) -> Net-(J4-Pad1)
- R14 pad 2: Net-(J4-Pad1) -> Net-(J4-Pad2)
- R8 pad 1: Net-(IC2-Pad2) -> Net-(C3-Pad1)
- R8 pad 2: Net-(C3-Pad1) -> Net-(IC2-Pad2)
- R9 pad 1: GND -> Net-(IC2-Pad2)
- R9 pad 2: Net-(IC2-Pad2) -> GND
