File: Hardware/mainboard/main.sch (KiCad schematic (older format))
At the start: 39 parts, among them IC2 LM358D, IC3 MC34063AD, J1 Conn_01x02_Male, J4 Conn_01x03_Male, J5 Conn_01x02_Male, Q1 IRF840, Q2 BC859, Q3 BC848, Q4 BC848

Commit message: Add info about zener diode voltage (#89)
Parts:
- D4: value D_Zener -> 5V1
Changed lines of the file:
@@
 EESchema Schematic File Version 4
-EELAYER 29 0
+EELAYER 30 0
 EELAYER END
 $Descr User 13234 8268
@@
 P 8550 5000
 F 0 "D4" V 8504 5079 50  0000 L CNN
-F 1 "D_Zener" V 8595 5079 50  0000 L CNN
+F 1 "5V1" V 8595 5079 50  0000 L CNN
 F 2 "Diode_THT:D_A-405_P2.54mm_Vertical_KathodeUp" H 8550 5000 50  0001 C CNN
 F 3 "~" H 8550 5000 50  0001 C CNN
